File: Hardware/Eagle/sdmapper.brd (EAGLE design)
At the start: 100 x 64.7 mm, 39 parts, among them IC1 SST39VF020N, IC2 HM628512ASOP32, IC3 XC95144XL_TQ100, IC4 LM1117-3V3, IC5 LM1117-3V3, T1 BC858, T2 BC858, X1 25MHz

Commit message: Alterando PCB e gerbers para retirar o logo PalMal
Parts:
- removed U$2: (no value), logos_fabio:LOGO_PALMAL_SILK_200MIL
Changed lines of the file:
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@@
 </element>
 <element name="U$1" library="logos_fabio" package="LOGO_FABIO_SILK_400MIL" value="" x="37.7825" y="16.8275" smashed="yes"/>
-<element name="U$2" library="logos_fabio" package="LOGO_PALMAL_SILK_200MIL" value="" x="75.2475" y="13.6525" smashed="yes"/>
 </elements>
 <signals>
